Commit message: working hexa_x_tilt model

File: models/hexa_x_tilt/hexa_x_tilt.urdf (robot description, URDF)
Before this commit: robot hexa_x_tilt, 13 links, 12 joints
Links:
- removed link hexa_x_tilt__cgo3_horizontal_arm_link
- removed link hexa_x_tilt__cgo3_mount_link
- removed link hexa_x_tilt__cgo3_vertical_arm_link
Joints:
- removed joint hexa_x_tilt__cgo3_horizontal_arm_joint
- removed joint hexa_x_tilt__cgo3_mount_joint
- removed joint hexa_x_tilt__cgo3_vertical_arm_joint
